File: hardware_scurity.kicad_pcb (KiCad board)
At the start: 2 copper layers, 137.3 x 121 mm, 34 parts, among them J10 Screw_Terminal_01x02, J11 Conn_01x04, J12 281740-4, J13 Conn_01x04, J14 Conn_01x01_Pin, J15 Screw_Terminal_01x02, J16 Screw_Terminal_01x02, J17 Screw_Terminal_01x02, J18 Screw_Terminal_01x02, J19 Screw_Terminal_01x02, J2 Conn_01x08, J20 Conn_01x02, J21 Conn_01x01_Pin, J22 Conn_01x08, J23 Conn_01x08, J24 Conn_01x01_Pin, J25 Jack-DC, J3 Conn_01x08, J4 Conn_01x02, J5 Conn_01x01_Pin, J6 Conn_01x04, J7 Conn_01x04, J8 Conn_01x01_Pin, J8 Screw_Terminal_01x02, J9 Conn_01x01_Pin, Q1 BF457, Q2 BF457

Commit message: fix(glitcher circuit): issue in glitcher circuit.
    change the design of glitcher circuit also change the cmos footprint
    as the old one was very big to set on the board.

Signed-off-by: tej-dabhankar <tejasdabhankar123@gmail.com>
Parts:
- added J1: Screw_Terminal_01x02, TerminalBlock:TerminalBlock_Altech_AK300-2_P5.00mm, F.Cu at (160.0, 73.3)
- added J26: Screw_Terminal_01x02, TerminalBlock:TerminalBlock_Altech_AK300-2_P5.00mm, F.Cu at (142.3, 136.9)
- added J28: Screw_Terminal_01x02, TerminalBlock:TerminalBlock_Altech_AK300-2_P5.00mm, F.Cu at (160.0, 84.8)
- J20: value Conn_01x02 -> Screw_Terminal_01x02; footprint Connector_PinSocket_2.54mm:PinSocket_1x02_P2.54mm_Vertical -> TerminalBlock:TerminalBlock_Altech_AK300-2_P5.00mm
- J4: value Conn_01x02 -> Conn_01x01_Pin; footprint Connector_PinSocket_2.54mm:PinSocket_1x02_P2.54mm_Vertical -> Connector_PinSocket_2.54mm:PinSocket_1x01_P2.54mm_Vertical
- Q1, Q2: value BF457 -> NMOS; footprint Package_TO_SOT_THT:TO-126-3_Vertical -> temmp:DIO_BAV99W_RFG
- moved J20 59.1 mm to (86.3, 131.3), turned to -90 degrees
- moved Q1 28.7 mm to (139.0, 50.8), turned to -90 degrees
- moved J4 20.3 mm to (78.0, 113.6)
- moved Q2 17.2 mm to (140.1, 80.8), turned to 180 degrees
- moved R4 13.7 mm to (111.8, 59.1)
- moved R3 6.19 mm to (117.7, 59.2), turned to 90 degrees
Connections:
- J15 pad 1: Net-(J15-Pin_1) -> Net-(J1-Pin_1)
- J15 pad 2: GND -> Net-(J1-Pin_2)
- J16 pad 1: Net-(J15-Pin_1) -> Net-(J1-Pin_1)
- J16 pad 2: GND -> Net-(J1-Pin_2)
- J17 pad 1: Net-(J15-Pin_1) -> Net-(J1-Pin_1)
- J17 pad 2: GND -> Net-(J1-Pin_2)
- J18 pad 1: Net-(J15-Pin_1) -> unconnected-(J18-Pin_1-Pad1)
- J18 pad 2: GND -> unconnected-(J18-Pin_2-Pad2)
- J19 pad 1: Net-(J15-Pin_1) -> unconnected-(J19-Pin_1-Pad1)
- J19 pad 2: GND -> unconnected-(J19-Pin_2-Pad2)
- J20 pad 1: Net-(J10-Pin_1) -> Net-(J1-Pin_1)
- J20 pad 2: Net-(J20-Pin_2) -> Net-(J1-Pin_2)
- J24 pad 1: Net-(J20-Pin_2) -> GND
- J25 pad 1: Net-(J15-Pin_1) -> Net-(Q1-D)
- J25 pad 2: GND -> Net-(J1-Pin_2)
- J3 pad 1: Net-(J20-Pin_2) -> GND
- J3 pad 2: Net-(J20-Pin_2) -> GND
- J3 pad 3: Net-(J20-Pin_2) -> GND
- J3 pad 4: Net-(J20-Pin_2) -> GND
- J3 pad 5: Net-(J20-Pin_2) -> GND
- J3 pad 6: Net-(J20-Pin_2) -> GND
- J3 pad 7: Net-(J20-Pin_2) -> GND
- J3 pad 8: Net-(J20-Pin_2) -> GND
- J4 pad 1: Net-(J15-Pin_1) -> Net-(J26-Pin_1)
- Q1 pad 1: GND -> Net-(Q1-D)
- Q1 pad 2: Net-(Q1-C) -> Net-(Q1-G)
- Q1 pad 3: Net-(J14-Pin_1) -> Net-(J1-Pin_1)
- Q2 pad 1: GND -> Net-(J26-Pin_1)
- Q2 pad 2: Net-(Q2-C) -> Net-(Q2-G)
- Q2 pad 3: Net-(J21-Pin_1) -> Net-(J10-Pin_1)
- R3 pad 1: Net-(J15-Pin_1) -> Net-(Q2-G)
- R3 pad 2: Net-(Q1-C) -> Net-(J21-Pin_1)
- R4 pad 1: Net-(J10-Pin_1) -> Net-(Q1-G)
- R4 pad 2: Net-(Q2-C) -> Net-(J14-Pin_1)
Routing:
- net GND: track 413.1 -> 39.6 mm
- net Net-(J1-Pin_2): track 0.00 -> 317.5 mm
- net Net-(J15-Pin_1): track 256.5 -> 0.00 mm
- net Net-(J1-Pin_1): track 0.00 -> 217.2 mm, vias 0 -> 1
- net Net-(J26-Pin_1): track 0.00 -> 124.2 mm, vias 0 -> 1
- net Net-(J20-Pin_2): track 117.5 -> 0.00 mm
- net Net-(J21-Pin_1): track 171.5 -> 77.7 mm
- net Net-(J10-Pin_1): track 138.5 -> 65.0 mm
- net Net-(Q2-G): track 0.00 -> 36.0 mm, vias 0 -> 2
- net Net-(Q1-G): track 0.00 -> 32.7 mm
- net Net-(J14-Pin_1): track 147.8 -> 120.6 mm
- net Net-(Q2-C): track 25.2 -> 0.00 mm
- net Net-(Q1-C): track 24.2 -> 0.00 mm
- net Net-(Q1-D): track 0.00 -> 22.9 mm, vias 0 -> 1
Other:
- board text removed: "gnd"
