File: hardware_scurity.kicad_sch (KiCad schematic)
At the start: 32 parts, among them J1 Raspberry_Pi_4, J10 Screw_Terminal_01x02, J11 Conn_01x04, J12 281740-4, J13 Conn_01x04, J14 Conn_01x01_Pin, J15 Screw_Terminal_01x02, J16 Screw_Terminal_01x02, J17 Screw_Terminal_01x02, J18 Screw_Terminal_01x02, J19 Screw_Terminal_01x02, J2 Conn_01x08, J20 Conn_01x02, J21 Conn_01x01_Pin, J22 Conn_01x08, J23 Conn_01x08, J24 Conn_01x01_Pin, J25 Jack-DC, J3 Conn_01x08, J4 Conn_01x02, J5 Conn_01x01_Pin, J6 Conn_01x04, J7 Conn_01x04, J8 Screw_Terminal_01x02, J9 Conn_01x01_Pin, Q1 BF457, Q2 BF457

Commit message: fix(glitcher circuit): issue in glitcher circuit.
    change the design of glitcher circuit also change the cmos footprint
    as the old one was very big to set on the board.

Signed-off-by: tej-dabhankar <tejasdabhankar123@gmail.com>
Parts:
- removed J1: Raspberry_Pi_4, footprint:MODULE_RASPBERRY_PI_4B_4GB, symbol Connector:Raspberry_Pi_4
- removed J20, J4: Conn_01x02, Connector_PinSocket_2.54mm:PinSocket_1x02_P2.54mm_Vertical, symbol Connector_Generic:Conn_01x02
- removed Q1, Q2: BF457, Package_TO_SOT_THT:TO-126-3_Vertical, symbol Transistor_BJT:BF457
- added J1, J20, J26, J28: Screw_Terminal_01x02, TerminalBlock:TerminalBlock_Altech_AK300-2_P5.00mm, symbol Connector:Screw_Terminal_01x02
- added J4: Conn_01x01_Pin, Connector_PinSocket_2.54mm:PinSocket_1x01_P2.54mm_Vertical, symbol Connector:Conn_01x01_Pin
- added Q1, Q2: NMOS, temmp:DIO_BAV99W_RFG, symbol Simulation_SPICE:NMOS
Connections:
- net GND: now also J24.1 (Pin_1), J3.1 (Pin_1), J3.2 (Pin_2), J3.3 (Pin_3), J3.4 (Pin_4), J3.5 (Pin_5), J3.6 (Pin_6), J3.7 (Pin_7), J3.8 (Pin_8), J26.2 (Pin_2); no longer J15.2 (Pin_2), J16.2 (Pin_2), J17.2 (Pin_2), J18.2 (Pin_2), J19.2 (Pin_2), J25.2
- net at R4.2: now also J14.1 (Pin_1)
- net at J21.1 (Pin_1): now also R3.2
- net at J10.1 (Pin_1), J8.1 (Pin_1): now also Q2.3 (S); no longer R4.1
- new net: J1.1 (Pin_1), J15.1 (Pin_1), J16.1 (Pin_1), J17.1 (Pin_1), J20.1 (Pin_1), J28.1 (Pin_1), Q1.3 (S)
- new net: J1.2 (Pin_2), J15.2 (Pin_2), J16.2 (Pin_2), J17.2 (Pin_2), J20.2 (Pin_2), J25.2, J28.2 (Pin_2)
- new net: J26.1 (Pin_1), J4.1 (Pin_1), Q2.1 (D)
- new net: J25.1, Q1.1 (D)
- new net: Q2.2 (G), R3.1
- new net: Q1.2 (G), R4.1
- now unconnected: J18.1 (Pin_1), J19.1 (Pin_1)
Other:
- moved on the sheet: J18, J19
